File: project_02/robot.sch (EAGLE design)
At the start: 26 parts, among them M1 RIGHT_MOTOR, M2 LEFT_MOTOR, SW1 PUSH_BUTTON, SW2 PUSH_BUTTON, U1 SERVO_SG90, U2 POCKETBEAGLE, U3 MOTOR_DRIVER_L293D, U4 TEMP_SENSOR_SI7021

Commit message: Schematic
Other:
- note added: "Change config-pin of P1_26 (GPIO I2C2 SDA) P1_28 (GPIO I2C2 SCL) to I2C"
- note added: "Change config-pin of P1_29 (GPIO 117) P1_30 (GPIO 43) P1_31 (GPIO 114) P1_32 (GPIO 42) P1_33 (GPIO 111) P1_34 (GPIO 26) to GPIO"
Changed lines of the file:
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@@
 <text x="330.2" y="93.98" size="5.08" layer="97">Mechanicals</text>
 <text x="157.48" y="154.94" size="1.778" layer="97">Temp: -40C : 125C</text>
+<text x="22.86" y="180.34" size="1.778" layer="97">Change config-pin of
+P1_29 (GPIO 117)
+P1_30 (GPIO 43)
+P1_31 (GPIO 114)
+P1_32 (GPIO 42)
+P1_33 (GPIO 111)
+P1_34 (GPIO 26)
+to GPIO</text>
+<text x="134.62" y="154.94" size="1.778" layer="97" align="bottom-right">Change config-pin of
+P1_26 (GPIO I2C2 SDA)
+P1_28 (GPIO I2C2 SCL)
+to I2C</text>
 </plain>
 <instances>
@@
 </drawing>
 <compatibility>
+<note version="6.3" minversion="6.2.2" severity="warning">
+Since Version 6.2.2 text objects can contain more than one line,
+which will not be processed correctly with this version.
+</note>
 <note version="9.0" severity="warning">
 Since Version 9.0, EAGLE supports the align property for labels.

Commit message: Schematic
Parts:
- U1: value SERVO_SG90 -> POCKETBEAGLE; device robot:SERVO_SG90 -> robot:POCKETBEAGLE
- U2: value POCKETBEAGLE -> MOTOR_DRIVER_L293D; device robot:POCKETBEAGLE -> robot:MOTOR_DRIVER_L293D
- U3: value MOTOR_DRIVER_L293D -> TEMP_SENSOR_SI7021; device robot:MOTOR_DRIVER_L293D -> robot:TEMP_SENSOR_SI7021
- U4: value TEMP_SENSOR_SI7021 -> SERVO_SG90; device robot:TEMP_SENSOR_SI7021 -> robot:SERVO_SG90
Connections:
- net BLUE_BUTTON: now also R1.1, U1B.GPIO_57; no longer R2.1, U2B.GPIO_57
- net BLUE_LED: now also U1B.GPIO_60; no longer U2B.GPIO_60
- net DRIVER_1,2EN: now also U1B.GPIO_111, U2.1,2EN; no longer U2B.GPIO_111, U3.1,2EN
- net DRIVER_1A: now also U1B.GPIO_114, U2.1A; no longer U2B.GPIO_114, U3.1A
- net DRIVER_1Y: now also U2.1Y; no longer U3.1Y
- net DRIVER_2A: now also U1B.GPIO_117, U2.2A; no longer U2B.GPIO_117, U3.2A
- net DRIVER_2Y: now also U2.2Y; no longer U3.2Y
- net DRIVER_3,4EN: now also U1B.GPIO_43, U2.3,4EN; no longer U2B.GPIO_43, U3.3,4EN
- net DRIVER_3A: now also U1B.GPIO_42, U2.3A; no longer U2B.GPIO_42, U3.3A
- net DRIVER_3Y: now also U2.3Y; no longer U3.3Y
- net DRIVER_4A: now also U1B.GPIO_26, U2.4A; no longer U2B.GPIO_26, U3.4A
- net DRIVER_4Y: now also U2.4Y; no longer U3.4Y
- net GND: now also U1A.GND_2, U1A.GND_3, U2.GND; no longer U1.GND, U2A.GND_2, U2A.GND_3, U2A.GND_USB1
- net SERVO: now also U1B.PWM0, U4.PWM; no longer U1.PWM, U2B.PWM0
- net TEMP_SEN_SCL: now also R4.1, U1B.I2C2_SCL, U3.SCL; no longer R3.1, U2B.I2C2_SCL, U4.SCL
- net TEMP_SEN_SDA: now also R3.1, U1B.I2C2_SDA, U3.SDA; no longer R4.1, U2B.I2C2_SDA, U4.SDA
- net VDD_3P3V: now also U1A.3.3V, U3.VDD; no longer U2A.3.3V, U4.VDD
- net VDD_5V: now also U1A.VOUT, U2.VCC, U4.PWR; no longer U1.PWR, U2A.VIN_USB1, U2A.VOUT, U3.VCC
- net YELLOW_BUTTON: now also R2.1, U1B.GPIO_59; no longer R1.1, U2B.GPIO_59
- net YELLOW_LED: now also U1B.GPIO_58; no longer U2B.GPIO_58
Other:
- note added: "P1_07 and P1_15 are unused pins"
- moved on the sheet: R1, R2, R3, R4
