File: project_02/robot.brd (EAGLE design)
At the start: 160 x 100 mm, 26 parts, among them M1 RIGHT_MOTOR, M2 LEFT_MOTOR, SW1 PUSH_BUTTON, SW2 PUSH_BUTTON, U1 SERVO_SG90, U2 POCKETBEAGLE, U3 MOTOR_DRIVER_L293D, U4 TEMP_SENSOR_SI7021

Commit message: Board
Parts:
- moved U3 234.4 mm to (63.5, 23.5), flipped to the bottom
- moved U4 224.1 mm to (36.2, 22.9)
- moved FUD6 208.3 mm to (63.5, 43.2)
- moved U2 208.2 mm to (1.27, 40.6), flipped to the bottom, turned to 180 degrees
- moved FUD2 202.3 mm to (63.5, 43.2), flipped to the bottom
- moved MGT1 193.9 mm to (68.6, 43.2)
- moved R5 186.0 mm to (61.0, 3.81), flipped to the bottom
- moved MGT4 183.3 mm to (68.6, 3.81)
- moved FUD4 164.5 mm to (8.89, 43.2)
- moved R2 161.3 mm to (48.3, 27.9)
- moved FUD1 159.0 mm to (8.89, 43.2), flipped to the bottom
- moved R1 145.7 mm to (24.1, 27.9)
- moved MGT2 144.6 mm to (3.81, 43.2)
- moved C1 140.4 mm to (36.3, 17.8)
- moved FUD5 139.5 mm to (8.89, 3.81)
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Routing:
- net BLUE_BUTTON: track 0.00 -> 91.9 mm
- net DRIVER_2A: track 0.00 -> 60.8 mm
- net DRIVER_1A: track 0.00 -> 43.5 mm
- net BLUE_LED: track 0.00 -> 40.0 mm
- net DRIVER_1,2EN: track 0.00 -> 37.5 mm
- net YELLOW_BUTTON: track 0.00 -> 35.0 mm
- net DRIVER_3,4EN: track 0.00 -> 30.9 mm
- net DRIVER_3A: track 0.00 -> 27.3 mm
- net DRIVER_3Y: track 0.00 -> 22.2 mm
- net YELLOW_LED: track 0.00 -> 21.0 mm
- net DRIVER_1Y: track 0.00 -> 20.7 mm
- net TEMP_SEN_SDA: track 0.00 -> 17.5 mm
- net DRIVER_4A: track 0.00 -> 13.2 mm
- net TEMP_SEN_SCL: track 0.00 -> 12.5 mm
- net DRIVER_4Y: track 0.00 -> 12.3 mm
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- added copper zone on layer 1, net CGND
- added copper zone on layer 16, net CGND
- added copper zone on layer 2, net GND
- added copper zone on layer 15, net VDD_3P3V
- added copper zone on layer 15, net VDD_5V
Other:
- board size 160 x 100 mm -> 72.4 x 47 mm
- board text added: "Blue"
- board text added: "ENGI 301"
- board text added: "For Drawing"
- board text added: "For Sensor"
- board text added: "LEFT"
- board text added: "Mood-Drawing Robot"
- board text added: "REV 1.0"
- board text added: "RIGHT"
- board text added: "Yellow"

Commit message: Board
Parts:
- added U$1: (no value), robot:LOGO
- U1: value SERVO_SG90 -> POCKETBEAGLE; device robot:SERVO -> robot:POCKETBEAGLE
- U2: value POCKETBEAGLE -> MOTOR_DRIVER_L293D; device robot:POCKETBEAGLE -> robot:MOTOR_DRIVER
- U3: value MOTOR_DRIVER_L293D -> TEMP_SENSOR_SI7021; device robot:MOTOR_DRIVER -> robot:TEMP_SENSOR
- U4: value TEMP_SENSOR_SI7021 -> SERVO_SG90; device robot:TEMP_SENSOR -> robot:SERVO
- moved FUD5 67.3 mm to (63.5, 43.2)
- moved FUD6 67.3 mm to (8.89, 3.81), flipped to the bottom
- moved U2 64.5 mm to (63.5, 23.5), turned to 0 degrees
- moved U1 53.4 mm to (1.27, 40.6), turned to 180 degrees
- moved U3 27.3 mm to (36.2, 22.9), flipped to the top
- moved U4 27.0 mm to (54.6, 42.5), flipped to the bottom, turned to 90 degrees
- moved R1 24.1 mm to (48.3, 27.9)
- moved R2 24.1 mm to (24.1, 27.9)
- moved R3 11.4 mm to (30.5, 27.9)
- moved R4 11.4 mm to (41.9, 27.9)
- flipped FUD1 to the top
- flipped FUD3 to the top
- flipped FUD4 to the bottom
Connections:
- new net VIN_USB1: U1.P1_07
- net BLUE_BUTTON: now also R1.1, U1.P2_06; no longer R2.1, U2.P2_06
- net BLUE_LED: now also U1.P2_08; no longer U2.P2_08
- net DRIVER_1,2EN: now also U1.P1_33, U2.1; no longer U2.P1_33, U3.1
- net DRIVER_1A: now also U1.P1_31, U2.2; no longer U2.P1_31, U3.2
- net DRIVER_1Y: now also M1.1, U2.3; no longer M1.PWR, U3.3
- net DRIVER_2A: now also U1.P1_29, U2.7; no longer U2.P1_29, U3.7
- net DRIVER_2Y: now also M1.2, U2.6; no longer M1.GND, U3.6
- net DRIVER_3,4EN: now also U1.P1_30, U2.9; no longer U2.P1_30, U3.9
- net DRIVER_3A: now also U1.P1_32, U2.10; no longer U2.P1_32, U3.10
- net DRIVER_3Y: now also M2.2, U2.11; no longer M2.GND, U3.11
- net DRIVER_4A: now also U1.P1_34, U2.15; no longer U2.P1_34, U3.15
- net DRIVER_4Y: now also M2.1, U2.14; no longer M2.PWR, U3.14
- net GND: now also U1.P1_16, U1.P1_22, U2.12, U2.13, U2.4, U2.5, U3.2, U4.3; no longer U1.3, U2.P1_15, U2.P1_16, U2.P1_22, U3.12, U3.13, U3.4, U3.5, U4.2
- net SERVO: now also U1.P1_36, U4.1; no longer U1.1, U2.P1_36
- net TEMP_SEN_SCL: now also R4.1, U1.P1_28, U3.4; no longer R3.1, U2.P1_28, U4.4
- net TEMP_SEN_SDA: now also R3.1, U1.P1_26, U3.1; no longer R4.1, U2.P1_26, U4.1
- net VDD_3P3V: now also U1.P1_14, U3.5; no longer U2.P1_14, U4.5
- net VDD_5V: now also U1.P1_24, U2.16, U2.8, U4.2; no longer U1.2, U2.P1_07, U2.P1_24, U3.16, U3.8
- net YELLOW_BUTTON: now also R2.1, U1.P2_02; no longer R1.1, U2.P2_02
- net YELLOW_LED: now also U1.P2_04; no longer U2.P2_04
Other:
- board text added: "U2"
- board text added: "U3"
